File: Schematics/RGBLedCube.kicad_sch (KiCad schematic)
At the start: 67 parts, among them J1 Conn_01x08_Pin, J10 Conn_01x08_Pin, J11 Conn_01x08_Pin, J12 Conn_01x08_Pin, J13 Conn_01x08_Pin, J14 Conn_01x08_Pin, J15 Conn_01x08_Pin, J16 Conn_01x08_Pin, J17 Conn_01x08_Pin, J18 Conn_01x08_Pin, J19 Conn_01x08_Pin, J2 Conn_01x08_Pin, J20 Conn_01x08_Pin, J21 Conn_01x08_Pin, J22 Conn_01x08_Pin, J23 Conn_01x08_Pin, J24 Conn_01x08_Pin, J25 Conn_01x08_Pin, J3 Conn_01x08_Pin, J4 Conn_01x08_Pin, J5 Conn_01x08_Pin, J6 Conn_01x08_Pin, J7 Conn_01x08_Pin, J8 Conn_01x08_Pin, J9 Conn_01x08_Pin, Q1 BC557, Q2 BC557, Q3 BC557, Q4 BC557, Q5 BC557, Q6 BC557, Q7 BC557, Q8 BC557, U1 74HC595, U10 74HC595, U11 74HC595, U12 74HC595, U13 74HC595, U14 74HC595, U15 74HC595, U16 74HC595, U17 74HC595, U18 74HC595, U19 74HC595, U2 74HC595, U20 74HC595, U21 74HC595, U22 74HC595, U23 74HC595, U24 74HC595, U25 74HC595, U3 74HC595, U4 74HC595, U5 74HC595, U6 74HC595, U7 74HC595, U8 74HC595, U9 74HC595

Commit message: Add schematics
Tracking-Id: EIP
Parts:
- J1, J10, J11, J12, J13, J14, J15, J16, J17, J18, J19, J2, J20, J21, J22, J23, J24, J25, J3, J4, J5, J6, J7, J8, J9: footprint (none) -> Connector_PinHeader_2.54mm:PinHeader_1x08_P2.54mm_Vertical
- R1, R2, R3, R4, R5, R6, R7, R8: footprint (none) -> Resistor_THT:R_Axial_DIN0414_L11.9mm_D4.5mm_P15.24mm_Horizontal
- U1, U10, U11, U12, U13, U14, U15, U16, U17, U18, U19, U2, U20, U21, U22, U23, U24, U25, U3, U4, U5, U6, U7, U8, U9: footprint (none) -> Package_DIP:DIP-16_W7.62mm
Connections:
- net at U10.10 (~{SRCLR}), U11.10 (~{SRCLR}), U12.10 (~{SRCLR})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: now also A1.27 (+5V), U1.10 (~{SRCLR}), U1.16 (VCC), U10.16 (VCC), U11.16 (VCC), U12.16 (VCC), U13.16 (VCC), U14.16 (VCC), U15.16 (VCC), U16.16 (VCC), U17.10 (~{SRCLR}), U17.16 (VCC), U18.10 (~{SRCLR}), U18.16 (VCC), U19.10 (~{SRCLR}), U19.16 (VCC), U2.10 (~{SRCLR}), U2.16 (VCC), U20.10 (~{SRCLR}), U20.16 (VCC), U21.10 (~{SRCLR}), U21.16 (VCC), U22.10 (~{SRCLR}), U22.16 (VCC), U23.10 (~{SRCLR}), U23.16 (VCC), U24.10 (~{SRCLR}), U24.16 (VCC), U25.10 (~{SRCLR}), U25.16 (VCC), U3.10 (~{SRCLR}), U3.16 (VCC), U4.10 (~{SRCLR}), U4.16 (VCC), U5.10 (~{SRCLR}), U5.16 (VCC), U6.10 (~{SRCLR}), U6.16 (VCC), U7.10 (~{SRCLR}), U7.16 (VCC), U8.10 (~{SRCLR}), U8.16 (VCC), U9.16 (VCC); no longer A1.8 (D5)
- net at J9.2 (Pin_2), U9.1 (QB): no longer U9.15 (QA)
- net at J17.1 (Pin_1): now also U17.15 (QA)
- net at J17.2 (Pin_2), U17.1 (QB): no longer U17.15 (QA)
- net at J1.1 (Pin_1): now also U1.15 (QA)
- net at J1.2 (Pin_2), U1.1 (QB): no longer U1.15 (QA)
- net at J9.1 (Pin_1): now also U9.15 (QA)
- new net: A1.8 (D5), U10.11 (SRCLK), U11.11 (SRCLK), U12.11 (SRCLK), U13.11 (SRCLK), U14.11 (SRCLK), U15.11 (SRCLK), U16.11 (SRCLK), U9.11 (SRCLK)
- new net: A1.5 (D2), U17.11 (SRCLK), U18.11 (SRCLK), U19.11 (SRCLK), U20.11 (SRCLK), U21.11 (SRCLK), U22.11 (SRCLK), U23.11 (SRCLK), U24.11 (SRCLK)
- new net: A1.10 (D7), U1.11 (SRCLK), U2.11 (SRCLK), U3.11 (SRCLK), U4.11 (SRCLK), U5.11 (SRCLK), U6.11 (SRCLK), U7.11 (SRCLK), U8.11 (SRCLK)
